File: eagle/half.sch (EAGLE design)
At the start: 116 parts, among them J3 AUDIO_JACK_TRRSSMD_RA, J5 AUDIO_JACK_TRRSSMD_RA

Commit message: update
Parts:
- added J10, J7, J8, J9: AUDIO_JACK_TRRSSMD_RA, SparkFun-Connectors:AUDIO_JACK_TRRSSMD_RA
- U$1, U$10, U$11, U$12, U$14, U$15, U$16, U$17, U$18, U$2, U$20, U$21, U$22, U$23, U$24, U$25, U$26, U$28, U$3, U$30, U$34, U$4, U$5, U$7, U$8, U$9: value CHERRY-MXSYMMETRIC -> CHERRY-MXSYMM-NOSILK; device cherrymx:CHERRY-MXSYMMETRIC -> cherrymx:CHERRY-MXSYMM-NOSILK
Connections:
- removed net 16: JP3.1
- removed net 2: JP3.5, R1.1
- new net 6: JP3.6
- new net 7: JP3.7
- new net N$36: J10.RING1, J7.RING1, J8.RING1, J9.RING1
- new net N$43: J10.TIP, J7.TIP, J8.TIP, J9.TIP
- new net N$44: J10.RING2, J7.RING2, J8.RING2, J9.RING2
- net 13: now also R1.1
- net GND: now also J10.EARTH, J7.EARTH, J8.EARTH, J9.EARTH
- net R4: now also JP3.5; no longer JP3.7
- net R5: now also JP3.1; no longer JP3.6
Other:
- note added: "Audio passthrough"
- note added: "assumes symmetric connection (tip -> tip)"

Commit message: updated PCB
Parts:
- added J12: (no value), SparkFun-Connectors:CONN_05NO_SILK
- added LED23, LED24, LED25, LED26, LED27, LED28, LED29, LED30, LED31, LED32, LED33, LED34, LED35, LED36, LED37, LED38, LED39, LED40, LED41, LED42, LED43, LED44: WS2812B_5050N, adafruit:WS2812B_5050N
- added R2: 330, adafruit:R-US_0204/7
- J2: device SparkFun-Connectors:CONN_041.27MM -> SparkFun-Connectors:CONN_05NO_SILK_SMALL
- J3, J5: value AUDIO_JACK_TRRSSMD_RA -> (none); device SparkFun-Connectors:AUDIO_JACK_TRRSSMD_RA -> SparkFun-Connectors:USB_MICRO-BUSB-B-MICRO-SMD-HOLES
Connections:
- removed net 12: J1.13
- removed net 14: J1.12
- removed net 25: J1.9
- removed net 26: J1.10
- removed net 27: J1.11
- removed net 34: J1.7
- removed net 35: J1.8
- new net 32: J1.5
- new net 33: J1.6
- new net 36: J1.1
- new net 37: J1.2
- new net 38: J1.3
- new net 39: J1.4
- new net N$45: J10.EARTH, J7.EARTH, J8.EARTH, J9.EARTH
- new net N$46: LED30.DI, LED39.DO
- new net N$47: LED24.DI, LED34.DO
- new net N$62: LED23.DI, R2.2
- new net N$63: LED24.DO, LED25.DI
- new net N$64: LED25.DO, LED26.DI
- new net N$65: LED26.DO, LED27.DI
- new net N$66: LED27.DO, LED28.DI
- new net N$67: LED28.DO, LED29.DI
- new net N$68: LED30.DO, LED31.DI
- new net N$69: LED31.DO, LED32.DI
- new net N$70: LED32.DO, LED33.DI
- new net N$71: LED33.DO, LED34.DI
- new net N$72: LED35.DI, LED44.DO
- new net N$73: LED35.DO, LED36.DI
- new net N$74: LED36.DO, LED37.DI
- new net N$75: LED37.DO, LED38.DI
- new net N$76: LED38.DO, LED39.DI
- new net N$77: LED23.DO, LED40.DI
- new net N$78: LED40.DO, LED41.DI
- new net N$79: LED41.DO, LED42.DI
- new net N$80: LED42.DO, LED43.DI
- new net N$81: LED43.DO, LED44.DI
- net +3V3: no longer J2.2, J3.RING1, J5.RING1
- net 4: now also R2.1
- net C1: now also J1.13; no longer J1.6
- net C2: now also J1.8; no longer J1.4
- net C3: now also J1.9; no longer J1.2
- net C4: now also J1.10; no longer J1.1
- net C5: now also J1.11; no longer J1.3
- net C6: now also J1.12; no longer J1.5
- net C7: now also J1.7
- net GND: now also J12.1, J3.GND, J5.GND, LED23.GND, LED24.GND, LED25.GND, LED26.GND, LED27.GND, LED28.GND, LED29.GND, LED30.GND, LED31.GND, LED32.GND, LED33.GND, LED34.GND, LED35.GND, LED36.GND, LED37.GND, LED38.GND, LED39.GND, LED40.GND, LED41.GND, LED42.GND, LED43.GND, LED44.GND; no longer J10.EARTH, J3.EARTH, J5.EARTH, J7.EARTH, J8.EARTH, J9.EARTH
- net SCL: now also J12.4, J2.4, J3.D+, J5.D+; no longer J2.3, J3.RING2, J5.RING2
- net SDA: now also J12.5, J2.5, J3.ID, J5.ID; no longer J2.4, J3.TIP, J5.TIP
- net VBAT: now also J12.2, J2.2, J3.VBUS, J5.VBUS, LED23.VDD, LED24.VDD, LED25.VDD, LED26.VDD, LED27.VDD, LED28.VDD, LED29.VDD, LED30.VDD, LED31.VDD, LED32.VDD, LED33.VDD, LED34.VDD, LED35.VDD, LED36.VDD, LED37.VDD, LED38.VDD, LED39.VDD, LED40.VDD, LED41.VDD, LED42.VDD, LED43.VDD, LED44.VDD
- net VUSB: now also J12.3, J2.3, J3.D-, J5.D-

Commit message: pcb update
Parts:
- removed J6: (no value), SparkFun-Connectors:CONN_024UCON-15767
- added J11: (no value), SparkFun-Connectors:JST_2MM_MALE
- J4: device SparkFun-Connectors:CONN_024UCON-15767 -> SparkFun-Connectors:JST_2MM_MALE
Connections:
- removed net 32: J1.5
- removed net 33: J1.6
- new net 34: J1.7
- new net 35: J1.8
- net C2: now also J1.6; no longer J1.8
- net C7: now also J1.5; no longer J1.7
- net GND: now also J11.-, J4.-; no longer J4.1, J6.1
- net SDA: now also J3.D-, J5.D-; no longer J3.ID, J5.ID
- net VBAT: now also J11.+, J3.ID, J4.+, J5.ID; no longer J3.VBUS, J4.2, J5.VBUS, J6.2
- net VUSB: now also J3.VBUS, J5.VBUS; no longer J3.D-, J5.D-
