File: eagle/half.brd (EAGLE design)
At the start: 138.2 x 89.8 mm, 116 parts, among them J3 AUDIO_JACK_TRRSSMD_RA, J5 AUDIO_JACK_TRRSSMD_RA

Commit message: update
Parts:
- added J10, J7, J8, J9: AUDIO_JACK_TRRSSMD_RA, SparkFun-Connectors:AUDIO_JACK_3.5MM_TRRS_SMD_RA
- U$1, U$10, U$11, U$12, U$14, U$15, U$16, U$17, U$18, U$2, U$20, U$21, U$22, U$23, U$24, U$25, U$26, U$28, U$3, U$30, U$34, U$4, U$5, U$7, U$8, U$9: value CHERRY-MXSYMMETRIC -> CHERRY-MXSYMM-NOSILK; device cherrymx:CHERRY-MX-SYMM -> cherrymx:CHERRY-MX-SYMM-NOSILK
- moved LED17 80.4 mm to (33.5, 55.3)
- moved LED13 80.4 mm to (113.8, 55.3)
- moved LED14 38.4 mm to (92.5, 55.3)
- moved LED16 38.3 mm to (54.2, 55.3)
- moved J5 25.6 mm to (138.6, 75.8), turned to 180 degrees
- moved J3 23.5 mm to (138.6, 75.8), turned to 0 degrees
- moved J6 19.4 mm to (124.7, 56.6)
- moved J4 19.4 mm to (124.7, 56.6)
- moved D6 17.0 mm to (119.0, 87.0)
- moved D15 16.7 mm to (8.49, 47.0)
- moved JP3 12.7 mm to (26.7, 59.7)
- moved D2 9.49 mm to (47.5, 78.7), turned to 0 degrees
- moved R1 3.92 mm to (15.8, 78.2)
- moved LED21 2.08 mm to (101.5, 74.4)
- moved LED18 2.08 mm to (44.5, 74.4)
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Connections:
- removed net 16: JP3.1
- removed net 2: JP3.5, R1.1
- new net 6: JP3.6
- new net 7: JP3.7
- new net N$36: J10.RING1, J7.RING1, J8.RING1, J9.RING1
- new net N$43: J10.TIP, J7.TIP, J8.TIP, J9.TIP
- new net N$44: J10.RING2, J7.RING2, J8.RING2, J9.RING2
- net 13: now also R1.1
- net GND: now also J10.EARTH, J7.EARTH, J8.EARTH, J9.EARTH
- net R4: now also JP3.5; no longer JP3.7
- net R5: now also JP3.1; no longer JP3.6
Routing:
- net N$44: track 0.00 -> 164.2 mm, vias 0 -> 3
- net N$43: track 0.00 -> 160.9 mm, vias 0 -> 3
- net N$36: track 0.00 -> 157.5 mm, vias 0 -> 3
- net N$33: track 0.00 -> 31.1 mm
- net N$35: track 0.00 -> 25.9 mm
- net N$42: track 0.00 -> 25.9 mm
- net N$34: track 0.00 -> 25.8 mm
- net N$39: track 0.00 -> 25.8 mm
- net N$58: track 0.00 -> 23.8 mm, vias 0 -> 2
- net SDA: track 177.2 -> 197.7 mm, vias 3 -> 4
- net N$37: track 0.00 -> 19.4 mm, vias 0 -> 2
- net N$40: track 0.00 -> 18.9 mm
- net R1: track 190.6 -> 171.9 mm, vias 2 -> 0
- net 2: track 18.5 -> 0.00 mm
- net N$61: track 0.00 -> 18.4 mm
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Other:
- outline, holes or cut-outs redrawn
- board text added: "+"
- board text added: "15"
- board text added: "18"
- board text added: "19"
- board text added: "2"
- board text added: "21"
- board text added: "23"
- board text added: "25"
- board text added: "26"
- board text added: "27"
- board text added: "3.3V"
- board text added: "32"
- board text added: "33"
- board text added: "34"
- board text added: "35"
- board text added: "36"
- board text added: "37"
- board text added: "38"
- board text added: "39"
- board text added: "5"
- board text added: "Audio"
- board text added: "GND"
- board text added: "RST"
- board text added: "RX"
- board text added: "TRRS pads not correct for digikey part"
- board text added: "TX"
- board text added: "VUSB"
- board text added: "left/right alignment of LEDs (could nudge ESP32 to the right a bit...)"
- board text removed: "Check fit of LEDs and TRRS jack by switches"
- board text removed: "NOTE: the position of this jack won't be symmetric across the board sides"
- board text removed: "SDA"
- board text removed: "Will LEDs fit between switches?"
- board text removed: "Will length of ESP32 fit? Its 2.320"x1""

Commit message: updated PCB
Parts:
- added J12: (no value), SparkFun-Connectors:1X05_NO_SILK
- added LED23, LED24, LED25, LED26, LED27, LED28, LED29, LED30, LED31, LED32, LED33, LED34, LED35, LED36, LED37, LED38, LED39, LED40, LED41, LED42, LED43, LED44: WS2812B_5050N, adafruit:WS2812B-NARROW
- added R2: 330, adafruit:0204/7
- J2: device SparkFun-Connectors:1X04_1.27MM -> SparkFun-Connectors:1X05_NO_SILK_SMALL
- J3, J5: value AUDIO_JACK_TRRSSMD_RA -> (none); device SparkFun-Connectors:AUDIO_JACK_3.5MM_TRRS_SMD_RA -> SparkFun-Connectors:USB-B-MICRO-SMD-HOLES
- moved J10 136.7 mm to (2.00, 18.9), turned to 180 degrees
- moved J9 136.7 mm to (2.00, 18.9), turned to 0 degrees
- moved D6 24.2 mm to (129.8, 65.4)
- moved D2 23.3 mm to (24.8, 84.2), turned to 270 degrees
- moved D3 16.0 mm to (78.5, 83.1)
- moved D29 13.9 mm to (8.06, 2.85), turned to 0 degrees
- moved D15 9.40 mm to (13.2, 55.1), turned to 0 degrees
- moved R1 7.96 mm to (8.63, 74.8)
- moved D20 6.23 mm to (127.9, 45.3)
- moved D8 6.03 mm to (7.87, 71.9), turned to 0 degrees
- moved D19 5.45 mm to (103.5, 45.0)
- moved D28 5.45 mm to (133.3, 26.3)
- moved D1 5.23 mm to (19.8, 83.4)
- moved J3 5.16 mm to (133.5, 76.5)
- moved J5 5.16 mm to (133.5, 76.5)
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Connections:
- removed net 12: J1.13
- removed net 14: J1.12
- removed net 25: J1.9
- removed net 26: J1.10
- removed net 27: J1.11
- removed net 34: J1.7
- removed net 35: J1.8
- new net 32: J1.5
- new net 33: J1.6
- new net 36: J1.1
- new net 37: J1.2
- new net 38: J1.3
- new net 39: J1.4
- new net N$45: J10.EARTH, J7.EARTH, J8.EARTH, J9.EARTH
- new net N$46: LED30.4-DIN, LED39.2-DOUT
- new net N$47: LED24.4-DIN, LED34.2-DOUT
- new net N$62: LED23.4-DIN, R2.2
- new net N$63: LED24.2-DOUT, LED25.4-DIN
- new net N$64: LED25.2-DOUT, LED26.4-DIN
- new net N$65: LED26.2-DOUT, LED27.4-DIN
- new net N$66: LED27.2-DOUT, LED28.4-DIN
- new net N$67: LED28.2-DOUT, LED29.4-DIN
- new net N$68: LED30.2-DOUT, LED31.4-DIN
- new net N$69: LED31.2-DOUT, LED32.4-DIN
- new net N$70: LED32.2-DOUT, LED33.4-DIN
- new net N$71: LED33.2-DOUT, LED34.4-DIN
- new net N$72: LED35.4-DIN, LED44.2-DOUT
- new net N$73: LED35.2-DOUT, LED36.4-DIN
- new net N$74: LED36.2-DOUT, LED37.4-DIN
- new net N$75: LED37.2-DOUT, LED38.4-DIN
- new net N$76: LED38.2-DOUT, LED39.4-DIN
- new net N$77: LED23.2-DOUT, LED40.4-DIN
- new net N$78: LED40.2-DOUT, LED41.4-DIN
- new net N$79: LED41.2-DOUT, LED42.4-DIN
- new net N$80: LED42.2-DOUT, LED43.4-DIN
- new net N$81: LED43.2-DOUT, LED44.4-DIN
- net +3V3: no longer J2.2, J3.RING1, J5.RING1
- net 4: now also R2.1
- net C1: now also J1.13; no longer J1.6
- net C2: now also J1.8; no longer J1.4
- net C3: now also J1.9; no longer J1.2
- net C4: now also J1.10; no longer J1.1
- net C5: now also J1.11; no longer J1.3
- net C6: now also J1.12; no longer J1.5
- net C7: now also J1.7
- net GND: now also J12.1, J3.GND, J5.GND, LED23.3-GND, LED24.3-GND, LED25.3-GND, LED26.3-GND, LED27.3-GND, LED28.3-GND, LED29.3-GND, LED30.3-GND, LED31.3-GND, LED32.3-GND, LED33.3-GND, LED34.3-GND, LED35.3-GND, LED36.3-GND, LED37.3-GND, LED38.3-GND, LED39.3-GND, LED40.3-GND, LED41.3-GND, LED42.3-GND, LED43.3-GND, LED44.3-GND; no longer J10.EARTH, J3.EARTH, J5.EARTH, J7.EARTH, J8.EARTH, J9.EARTH
- net SCL: now also J12.4, J2.4, J3.D+, J5.D+; no longer J2.3, J3.RING2, J5.RING2
- net SDA: now also J12.5, J2.5, J3.ID, J5.ID; no longer J2.4, J3.TIP, J5.TIP
- net VBAT: now also J12.2, J2.2, J3.VBUS, J5.VBUS, LED23.1-VDD, LED24.1-VDD, LED25.1-VDD, LED26.1-VDD, LED27.1-VDD, LED28.1-VDD, LED29.1-VDD, LED30.1-VDD, LED31.1-VDD, LED32.1-VDD, LED33.1-VDD, LED34.1-VDD, LED35.1-VDD, LED36.1-VDD, LED37.1-VDD, LED38.1-VDD, LED39.1-VDD, LED40.1-VDD, LED41.1-VDD, LED42.1-VDD, LED43.1-VDD, LED44.1-VDD
- net VUSB: now also J12.3, J2.3, J3.D-, J5.D-
Routing:
- net VUSB: track 0.00 -> 215.6 mm, vias 0 -> 4
- net +3V3: track 213.8 -> 0.00 mm, vias 4 -> 0
- net C7: track 36.3 -> 249.4 mm
- net VBAT: track 559.0 -> 710.9 mm, vias 9 -> 17
- net N$45: track 0.00 -> 108.1 mm, vias 0 -> 5
- net N$43: track 160.9 -> 102.8 mm
- net N$67: track 0.00 -> 48.9 mm
- net C2: track 146.4 -> 194.5 mm, vias 2 -> 3
- net N$72: track 0.00 -> 43.0 mm, vias 0 -> 2
- net N$80: track 0.00 -> 33.0 mm
- net N$81: track 0.00 -> 32.2 mm
- net N$73: track 0.00 -> 31.3 mm, vias 0 -> 4
- net N$27: track 11.2 -> 40.8 mm
- net N$66: track 0.00 -> 29.5 mm, vias 0 -> 2
- net N$76: track 0.00 -> 29.1 mm, vias 0 -> 2
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Other:
- board size 138.2 x 89.8 mm -> 135.6 x 90.2 mm
- board text added: """
- board text added: "/"
- board text added: "1"
- board text added: "3"
- board text added: "6"
- board text added: "7"
- board text added: "8"
- board text added: "9"
- board text added: ";"
- board text added: "<"
- board text added: ">"
- board text added: "A"
- board text added: "Alt"
- board text added: "Audio in"
- board text added: "Audio out"
- board text added: "B"
- board text added: "Back"
- board text added: "C"
- board text added: "Caps"
- board text added: "Ctrl"
- board text added: "D"
- board text added: "Del"
- board text added: "Down"
- board text added: "E"
- board text added: "Enter"
- board text added: "Esc"
- board text added: "Extra"
- board text added: "F"
- board text added: "G"
- board text added: "H"
- board text added: "I"
- board text added: "J"
- board text added: "K"
- board text added: "L"
- board text added: "Left"
- board text added: "M"
- board text added: "M3"
- board text added: "N"
- board text added: "NOTE: all switches, LEDs, diodes, resistor and capacitors go on one side of the board; all remaining IO (USB, pogopins and TRRS) go on the opposite side"
- board text added: "NOTE: the alignment pins for the springed male I2C connector will have to be drilled manually"
- board text added: "NOTE: the position of the TRRS ports will hit the alignment pins of the switches. There is no way around this since there isn't enough space between the switches; the workaround will be to trim off the excess pin stickout out of the PCB."
- board text added: "O"
- board text added: "P"
- board text added: "Q"
- board text added: "R"
- board text added: "Right"
- board text added: "S"
- board text added: "Shift"
- board text added: "Space"
- board text added: "T"
- board text added: "Tab"
- board text added: "U"
- board text added: "Up"
- board text added: "V"
- board text added: "W"
- board text added: "Win"
- board text added: "X"
- board text added: "Y"
- board text added: "Z"
- board text added: "[ ]"
- board text added: "top distance from edge of board to switches should be symmetric on top & bottom of board"
- board text added: "~"
- board text removed: "Audio"
- board text removed: "Mounting holes for board"
- board text removed: "Need to check symmetric fit and orientation of ESP32"
- board text removed: "TRRS pads not correct for digikey part"
- board text removed: "larger trace width for VBAT since it will carry LED current?"
- board text removed: "left/right alignment of LEDs (could nudge ESP32 to the right a bit...)"
- board text removed: "location of magnet I2C port?"
- board text removed: "side L"
- board text removed: "side R"

Commit message: pcb update
Parts:
- removed J6: (no value), SparkFun-Connectors:JST-2-SMD-VERT
- added J11: (no value), SparkFun-Connectors:JST-2-SMD
- J4: device SparkFun-Connectors:JST-2-SMD-VERT -> SparkFun-Connectors:JST-2-SMD
- moved R2 2.54 mm to (23.1, 77.7)
Connections:
- removed net 32: J1.5
- removed net 33: J1.6
- new net 34: J1.7
- new net 35: J1.8
- net C2: now also J1.6; no longer J1.8
- net C7: now also J1.5; no longer J1.7
- net GND: now also J11.1, J4.1; no longer J4.GND, J6.GND
- net SDA: now also J3.D-, J5.D-; no longer J3.ID, J5.ID
- net VBAT: now also J11.2, J3.ID, J4.2, J5.ID; no longer J3.VBUS, J4.VCC, J5.VBUS, J6.VCC
- net VUSB: now also J3.VBUS, J5.VBUS; no longer J3.D-, J5.D-
Routing:
- net SCL: track 184.1 -> 191.1 mm, vias 4 -> 5
- net C7: track 249.4 -> 244.0 mm
- net C2: track 194.5 -> 189.4 mm
- net 4: track 13.8 -> 16.4 mm
- net VBAT: track 710.9 -> 713.1 mm, vias 17 -> 16
- net VUSB: track 215.6 -> 214.8 mm, vias 4 -> 5
- net SDA: track 191.6 -> 191.8 mm, vias 4 -> 5

Commit message: v1 of pcb
Parts:
- moved D32 0.95 mm to (77.3, 8.33)
- moved D31 0.90 mm to (55.6, 8.48)
Routing:
- net N$7: track 27.0 -> 28.2 mm
- net C4: track 189.8 -> 190.6 mm
- net C3: track 172.7 -> 173.5 mm
- net C7: track 244.0 -> 243.3 mm
- net R5: track 140.6 -> 141.2 mm
Other:
- board text added: "TACOCAT v1"
- board text removed: "MOOCOW v1"
- board text removed: "top distance from edge of board to switches should be symmetric on top & bottom of board"
