File: PCB/half.sch (EAGLE design)
At the start: 144 parts, among them J10 AUDIO_JACK_TRRSSMD_RA, J7 AUDIO_JACK_TRRSSMD_RA, J8 AUDIO_JACK_TRRSSMD_RA, J9 AUDIO_JACK_TRRSSMD_RA

Commit message: PCB update, improved micro usb part with longer pads, capacitor added to VBAT circuit
Parts:
- added C17: 1000uF, adafruit:CPOL-USE3.5-8
- J3, J5: device SparkFun-Connectors:USB_MICRO-BUSB-B-MICRO-SMD-HOLES -> EAGLE-INPUT_OUTPUT_CONNECTORS-rev17a:629105136821
Connections:
- net GND: now also C17.-
- net VBAT: now also C17.+

Commit message: pcb update
Parts:
- J3, J5: value (none) -> USB_MINI-B_SMT; device EAGLE-INPUT_OUTPUT_CONNECTORS-rev17a:629105136821 -> SparkFun-Connectors:USB_MINI-B_SMT
- LED1, LED10, LED11, LED12, LED13, LED14, LED15, LED16, LED17, LED18, LED19, LED2, LED20, LED21, LED22, LED23, LED24, LED25, LED26, LED27, LED28, LED29, LED3, LED30, LED31, LED32, LED33, LED34, LED35, LED36, LED37, LED38, LED39, LED4, LED40, LED41, LED42, LED43, LED44, LED5, LED6, LED7, LED8, LED9: value WS2812B_5050N -> WS2812BLONGPADS; device adafruit:WS2812B_5050N -> adafruit:WS2812BLONGPADS
